File: PII4XE.kicad_sch (KiCad schematic)
At the start: 37 parts, among them Q5 2N7002, Q6 2N7002, Q8 2N7002, U17 SN74HC10DR-separate, U23 PIIX4_82371EB, U27 SN74HC112DR, U28 SN74LS07DR, U5 SN74LVC14A, Y2 SG-3030CM

Commit message: improved Cover Sheet, BLOCK DIAGRAM from PDF thru SVG import
Changed lines of the file:
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@@
 (kicad_sch
-	(version 20231120)
+	(version 20241004)
 	(generator "eeschema")
-	(generator_version "8.0")
+	(generator_version "8.99")
 	(paper "A2" portrait)
+	(title_block
+		(date "Thursday, April 09, 1998")
+		(rev "1.0")
+	)
+	(text "JP21 CONFIG.\n1-2	SAVE STATE ON POWER DOWN.\n2-3	PIIX4 POWERS ON SYS. AT POWER-UP."
+		(exclude_from_sim no)
+		(at 328.93 281.94 0)
+		(effects
+			(font
+				(size 1.27 1.27)
+			)
+			(justify left)
+		)
+	)
 	(junction
 		(at 266.7 457.2)
@@
 		)
 	)
-	(text "JP21 CONFIG.\n1-2	SAVE STATE ON POWER DOWN.\n2-3	PIIX4 POWERS ON SYS. AT POWER-UP."
-		(exclude_from_sim no)
-		(at 328.93 281.94 0)
-		(effects
-			(font
-				(size 1.27 1.27)
-			)
-			(justify left)
-		)
-	)
