File: Power Connector & Misc.kicad_sch (KiCad schematic)
At the start: 55 parts, among them J25 POWER LED, J26 Conn_01x03_Pin, J27 SPEAKER HEADER, J28 HDD LED, J29 Jumper_2_Open, J30 ATX-24, J39 Conn_01x03_Socket, Q2 2N3904, Q7 BSS84, U12 SN74LS07DR, U14 SN74LS07DR, U16 74AHC1G08, U17 SN74HC10DR-separate, U28 SN74LS07DR, U5 SN74LVC14A, U8 74HCT14

Commit message: improved Cover Sheet, BLOCK DIAGRAM from PDF thru SVG import
Other:
- title: (none) -> Power Connector & Misc
