File: 82443BX.kicad_sch (KiCad schematic)
At the start: 42 parts, among them U19 440BX CHIPSET, U20 CKBF

Commit message: improved Cover Sheet, BLOCK DIAGRAM from PDF thru SVG import
Changed lines of the file:
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@@
 (kicad_sch
-	(version 20231120)
+	(version 20241004)
 	(generator "eeschema")
-	(generator_version "8.0")
+	(generator_version "8.99")
 	(paper "A1")
+	(title_block
+		(date "Thursday, April 09, 1998")
+		(rev "1.0")
+	)
+	(text "R39 8.2K\nNOT NEEDED\n"
+		(exclude_from_sim no)
+		(at 386.334 25.146 0)
+		(effects
+			(font
+				(size 1.27 1.27)
+			)
+		)
+	)
+	(text "can't find  FBHS01L\nFairrite 2512066017Y1 used on other boards... \nBias Current (ma): 200 \nSize: 1206\nDC Resistance: 0.30\nImpedance@ 100MHz: 600\n"
+		(exclude_from_sim no)
+		(at 751.078 319.532 0)
+		(effects
+			(font
+				(size 1.27 1.27)
+			)
+		)
+	)
+	(text " **NOTE** Locate\n circuitry close to\n 443BX."
+		(exclude_from_sim no)
+		(at 439.166 551.688 0)
+		(effects
+			(font
+				(size 1.27 1.27)
+			)
+		)
+	)
+	(text "**Locate r280 close to CKBF and R281 close to 443BX.\n**Locate \"T\" and cap close to BX.\n** Please make DCLKREF trace length equal to 2.5\" more\n than the DCLK outputs to the DIMMs. DCLK outputs to\n the DIMMs should all be the same recommended length.\n Example: if DCLK[0-11] = 2.5\"\n then DCLKREF = 2.5\" + 2.5\".\n\n "
+		(exclude_from_sim no)
+		(at 690.118 503.682 0)
+		(effects
+			(font
+				(size 1.27 1.27)
+			)
+		)
+	)
 	(junction
 		(at 231.14 271.78)
@@
 		)
 	)
-	(text "R39 8.2K\nNOT NEEDED\n"
-		(exclude_from_sim no)
-		(at 386.334 25.146 0)
-		(effects
-			(font
-				(size 1.27 1.27)
-			)
-		)
-	)
-	(text "can't find  FBHS01L\nFairrite 2512066017Y1 used on other boards... \nBias Current (ma): 200 \nSize: 1206\nDC Resistance: 0.30\nImpedance@ 100MHz: 600\n"
-		(exclude_from_sim no)
-		(at 751.078 319.532 0)
-		(effects
-			(font
-				(size 1.27 1.27)
-			)
-		)
-	)
-	(text " **NOTE** Locate\n circuitry close to\n 443BX."
-		(exclude_from_sim no)
-		(at 439.166 551.688 0)
-		(effects
-			(font
-				(size 1.27 1.27)
-			)
-		)
-	)
-	(text "**Locate r280 close to CKBF and R281 close to 443BX.\n**Locate \"T\" and cap close to BX.\n** Please make DCLKREF trace length equal to 2.5\" more\n than the DCLK outputs to the DIMMs. DCLK outputs to\n the DIMMs should all be the same recommended length.\n Example: if DCLK[0-11] = 2.5\"\n then DCLKREF = 2.5\" + 2.5\".\n\n "
-		(exclude_from_sim no)
-		(at 690.118 503.682 0)
-		(effects
-			(font
-				(size 1.27 1.27)
-			)
-		)
-	)

Commit message: page 6,7,8 82443BX chipset, various small fixes
Parts:
- removed C6013: 0.001uF, Capacitor_SMD:C_0201_0603Metric, symbol Device:C
- removed L16: 600 25%, Inductor_SMD:L_1206_3216Metric, symbol Device:L
- removed R1187, R1188, R1189, R1190: 0, Resistor_SMD:R_0201_0603Metric, symbol Device:R
- removed R6021: 100, Resistor_SMD:R_0201_0603Metric, symbol Device:R
- removed R6022, R6025: 22, Resistor_SMD:R_0201_0603Metric, symbol Device:R
- removed R6023: 150 1%, Resistor_SMD:R_0201_0603Metric, symbol Device:R
- removed R6024: 100 1%, Resistor_SMD:R_0201_0603Metric, symbol Device:R
- removed R6026: 10K, Resistor_SMD:R_0201_0603Metric, symbol Device:R
- removed U19: 440BX CHIPSET, P2-3_ERA:440BX_Chipset_Generic, symbol P2-3_era:BXChipset
- added L16: FBHS01L, symbol Device:FerriteBead
- added R39: 8.2K, Resistor_SMD:R_0201_0603Metric, symbol Device:R
- added U19: 82443BX, P2-3_ERA:440BX_Chipset_Generic, symbol P2-3_era:440BX_Chipset
- C175, C177, C179, C181, C183: value 0.01uF -> .01uF
- R281: value 47 -> 22
- renumbered C6012 to C162
Connections:
- net ADS#: now also U19.K21 (ADS#)
- net BNR#: now also U19.H24 (BNR#)
- net BPRI#: now also U19.H26 (BPRI#)
- net BREQ0#: now also U19.B26 (BREQ0#)
- net BXHCLK: now also U19.N23 (HCLKIN)
- net CRESET#: now also U19.M26 (CRESET#)
- net CS_A#0: now also U19.AB14 (CSA0#/RASA0#)
- net CS_A#1: now also U19.AF15 (CSA1#/RASA1#)
- net CS_A#2: now also U19.AE15 (CSA2#/RASA2#)
- net CS_A#3: now also U19.AC15 (CSA3#/RASA3#)
- net CS_A#4: now also U19.AD15 (CSA4#/RASA4#)
- net CS_A#5: now also U19.AE16 (CSA5#/RASA5#)
- net CS_A#6: now also U19.AE24 (CSA6#/CKE2)
- net CS_A#7: now also U19.AD23 (CSA7#/CKE3)
- net CS_B#0: now also U19.AE25 (CSB0#/RASB0#)
- net CS_B#1: now also U19.AD24 (CSB1#/RASB1#)
- net CS_B#2: now also U19.AD26 (CSB2#/RASB2#)
- net CS_B#3: now also U19.AC24 (CSB3#/RASB3#)
- net CS_B#4: now also U19.AC26 (CSB4#/RASB4#)
- net CS_B#5: now also U19.AB23 (CSB5#/RASB5#)
- net CS_B#6: now also U19.AC23 (CKE4#/CSB6)
- net CS_B#7: now also U19.AF24 (CKE5#/CSB7)
- net DBSY#: now also U19.L23 (DBSY#)
- net DCLKREF: now also U19.AB22 (DCLKRD), U19.AD25 (DCLKWR)
- net DEFER#: now also U19.J26 (DEFER#)
- net DQMA0: now also U19.AD13 (DQMA0/CASA0#)
- net DQMA1: now also U19.AC13 (DQMA1/CASA1#)
- net DQMA2: now also U19.AC25 (DQMA2/CASA2#)
- net DQMA3: now also U19.AB26 (DQMA3/CASA3#)
- net DQMA4: now also U19.AE14 (DQMA4/CASA4#)
- net DQMA5: now also U19.AC14 (DQMA5/CASA5#)
- net DQMA6: now also U19.AA22 (DQMA6/CASA6#)
- net DQMA7: now also U19.AA24 (DQMA7/CASA7#)
- net DQMB1: now also U19.AE13 (DQMB1/CASB1#)
- net DQMB5: now also U19.AD14 (DQMB5/CASB5#)
- net DRDY#: now also U19.K23 (DRDY#)
- net FENA: now also U19.AC22 (CKE0/FENA)
- net GCKE: now also U19.AF23 (CKE1/GCKE)
- net HA#10: now also U19.G22 (HA10#)
- net HA#11: now also U19.F22 (HA11#)
- net HA#12: now also U19.F23 (HA12#)
- net HA#13: now also U19.F24 (HA13#)
- net HA#14: now also U19.F25 (HA14#)
- net HA#15: now also U19.E23 (HA15#)
- net HA#16: now also U19.E26 (HA16#)
- net HA#17: now also U19.E25 (HA17#)
- net HA#18: now also U19.D25 (HA18#)
- net HA#19: now also U19.D26 (HA19#)
- net HA#20: now also U19.B25 (HA20#)
- net HA#21: now also U19.C26 (HA21#)
- net HA#22: now also U19.A25 (HA22#)
- net HA#23: now also U19.C25 (HA23#)
- net HA#24: now also U19.A24 (HA24#)
- net HA#25: now also U19.D24 (HA25#)
- net HA#26: now also U19.C23 (HA26#)
- net HA#27: now also U19.B24 (HA27#)
- net HA#28: now also U19.C24 (HA28#)
- net HA#29: now also U19.A23 (HA29#)
- net HA#3: now also U19.G25 (HA3#)
- net HA#30: now also U19.E22 (HA30#)
- net HA#31: now also U19.D23 (HA31#)
- net HA#4: now also U19.H22 (HA4#)
- net HA#5: now also U19.G23 (HA5#)
- net HA#6: now also U19.H23 (HA6#)
- net HA#7: now also U19.G24 (HA7#)
- net HA#8: now also U19.F26 (HA8#)
- net HA#9: now also U19.G26 (HA9#)
- net HIT#: now also U19.L24 (HIT#)
- net HITM#: now also U19.L22 (HITM#)
- net HLOCK#: now also U19.K22 (HLOCK#)
- net HRESET#: now also U19.B23 (CPURST#)
- net HTRDY#: now also U19.H25 (HTRDY#)
- net MAA0: now also U19.AF17 (MAA0)
- net MAA1: now also U19.AB16 (MAA1)
- net MAA10: now also U19.AD20 (MAA10)
- net MAA11: now also U19.AF21 (MAA11)
- net MAA12: now also U19.AC21 (MAA12)
- net MAA13: now also U19.AF25 (MAA13)
- net MAA2: now also U19.AE17 (MAA2)
- net MAA3: now also U19.AC17 (MAA3)
- net MAA4: now also U19.AF18 (MAA4)
- net MAA5: now also U19.AE19 (MAA5)
- net MAA6: now also U19.AF19 (MAA6)
- net MAA7: now also U19.AC18 (MAA7)
- net MAA8: now also U19.AC19 (MAA8)
- net MAA9: now also U19.AE20 (MAA9)
- net MAB#0: now also U19.AD16 (MAB0#)
- net MAB#1: now also U19.AC16 (MAB1#)
- net MAB#10: now also U19.AB20 (MAB10)
- net MAB#11: now also U19.AE21 (MAB11#)
- net MAB#12: now also U19.AD21 (MAB12#)
- net MAB#13: now also U19.AF22 (MAB13)
- net MAB#2: now also U19.AD17 (MAB2#)
- net MAB#3: now also U19.AB17 (MAB3#)
- net MAB#4: now also U19.AE18 (MAB4#)
- net MAB#5: now also U19.AD19 (MAB5#)
- net MAB#6: now also U19.AB18 (MAB6#)
- net MAB#7: now also U19.AB19 (MAB7#)
- net MAB#8: now also U19.AF20 (MAB8#)
- net MAB#9: now also U19.AC20 (MAB9#)
- net PCIRST#: now also U19.A3 (PCIRST#)
- net SCAS_A#: now also U19.AF12 (SCAS_A#)
- net SCAS_B#: now also U19.AB13 (SCAS_B#)
- net SRAS_A#: now also U19.AF16 (SRAS_A#)
- net SRAS_B#: now also U19.AA17 (SRAS_B#)
- net WE_A#: now also U19.AE12 (WE_A#)
- net WE_B#: now also U19.AC12 (WE_B#)
- net at C174.1, C175.1, C176.1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: now also L16.2
- net GND: now reaches C174.2, C175.2, C176.2, C177.2, C178.2, C179.2, C180.2, C181.2, C182.2, C183.2, C184.2
- net GND: now also C162.2, U20.22 (VSS), U19.A1 (VSS), U19.A14 (VSS), U19.A26 (VSS), U19.C18 (VSS), U19.C22 (VSS), U19.C5 (VSS), U19.C9 (VSS), U19.E12 (VSS), U19.E15 (VSS), U19.E24 (VSS), U19.E3 (VSS), U19.F19 (VSS), U19.F21 (VSS), U19.F6 (VSS), U19.F8 (VSS), U19.H21 (VSS), U19.H6 (VSS), U19.J24 (VSS), U19.J3 (VSS)
- net at R281.1: now also U19.AB21 (DCLKO)
- net Earth: no longer names the net of U20.10 (VSS), U20.15 (VSS), U20.19 (VSS), U20.26 (VSSIIC), U20.27 (VSS), U20.30 (VSS), U20.34 (VSS), U20.39 (VSS), U20.43 (VSS), U20.6 (VSS)
- net Earth: no longer C162.2, U20.22 (VSS)
- new net: U19.AA18 (VDD), U19.AA20 (VDD), U19.AA7 (VDD), U19.AA9 (VDD), U19.F18 (VDD), U19.F20 (VDD), U19.F7 (VDD), U19.F9 (VDD), U19.G21 (VDD), U19.G6 (VDD), U19.J21 (VDD), U19.J6 (VDD), U19.V21 (VDD), U19.Y21 (VDD)
- new net: R39.1, U19.M25 (TESTIN#)
- new net HREQ#0: U19.J22 (HREQ#0)
- new net HREQ#1: U19.J23 (HREQ#1)
- new net HREQ#2: U19.K24 (HREQ#2)
- new net HREQ#3: U19.K25 (HREQ#3)
- new net HREQ#4: U19.J25 (HREQ#4)
- new net RS#0: U19.K26 (RS#0)
- new net RS#1: U19.L26 (RS#1)
- new net RS#2: U19.L25 (RS#2)
- no-connect marks 4 -> 5
Other:
- note added: "** TESTIN# pullup may be removed after validation has been completed."
- note added: "**Locate R280 close to CKBF and R281 close to 443BX. **Locate "T" and cap close to BX. ** Please make DCLKREF trace length equal to 2.5" more than the DCLK outputs to the DIMMs. DCLK outputs to the DIMMs should all be the same recommended length."
- note added: "**Please Note ** These clock assignments may not be optimum."
- note added: "*The unused SDRAM clocks may be disabled using the SMBus interface."
- note added: "Exam ple: if DCLK[0-11] = 2.5" then DCLKREF = 2.5" + 2.5""
- note added: "slave address = 1101001b"
- note removed: "**Locate r280 close to CKBF and R281 close to 443BX. **Locate "T" and cap close to BX. ** Please make DCLKREF trace length equal to 2.5" more than the DCLK outputs to the DIMMs. DCLK outputs to the DIMMs should all be the same recommended length. Example: if DCLK[0-11] = 2.5" then DCLKREF = 2.5" + 2.5"."
- note removed: "**NOTE** Locate circuitry close to 443BX."
- note removed: "R39 8.2K NOT NEEDED"
- note removed: "can't find FBHS01L Fairrite 2512066017Y1 used on other boards... Bias Current (ma): 200 Size: 1206 DC Resistance: 0.30 Impedance@ 100MHz: 600"
- title: (none) -> 82443BX SYSTEM AND DRAM INTERFACES
- moved on the sheet: C162, C174, C175, C176, C177, C178, C179, C180, C181, C182, C183, C184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
